Commit message: updated Physical representation of the map

File: urdf/avalanche_victim.xacro (robot description, xacro)
@@ -1,5 +1,5 @@
 <?xml version="1.0" ?>
-<robot name="rock" xmlns:xacro="http://ros.org/wiki/xacro">
-  <xacro:macro name="rock_macro" params="name fixed_frame *origin">
+<robot name="avalanche_victim" xmlns:xacro="http://ros.org/wiki/xacro">
+  <xacro:macro name="avalanche_victim_macro" params="name fixed_frame *origin">
     <gazebo>
       <static>true</static>
@@ -10,5 +10,5 @@
 	<origin rpy="0 0 0" xyz="0 0 0"/>
 	<geometry>
-	  <mesh filename="package://iai_outdoor_models/models/rock/Rock.dae"/>
+	  <mesh filename="package://iai_outdoor_models/models/avalanche_victim/victim.dae"/>
 	</geometry>
 <!--
@@ -16,5 +16,5 @@
 	-->
 <!--
-	<material name="IAI_RESCUE/rock">
+	<material name="IAI_RESCUE/avalanche_victim">
 	<color rgba="0.31 0.15 0.033 1.0"/>
       </material>
@@ -24,5 +24,5 @@
 	<origin rpy="0 0 0" xyz="0 0 0"/>
 	<geometry>
-	  <mesh filename="package://iai_outdoor_models/models/rock/Rock.stl"/>
+	  <mesh filename="package://iai_outdoor_models/models/avalanche_victim/victim.dae"/>
 	</geometry>
       </collision>

File: urdf/broad_leaved_tree.xacro (robot description, xacro)
@@ -28,10 +28,10 @@
     </inertial>
   </link>
-  <link name="broad_leaved_tree_branches">
+  <link name="${name}_branches">
     <!--MAIN_BODY-->
     <visual>
       <origin rpy="0 0 0" xyz="0 0 0"/>
       <geometry>
-        <mesh filename="package://iai_outdoor_models/models/broad_leaved_tree/broad_leaved_tree_branches.stl"/>
+        <mesh filename="package://iai_outdoor_models/models/broad_leaved_tree/broad_leaved_tree_leaves.stl"/>
       </geometry>
       <material name="IAI_RESCUE/broad_leaved_branch">
@@ -42,5 +42,5 @@
       <origin rpy="0 0 0" xyz="0 0 0"/>
       <geometry>
-        <mesh filename="package://iai_outdoor_models/models/broad_leaved_tree/broad_leaved_tree_branches.stl"/>
+        <mesh filename="package://iai_outdoor_models/models/broad_leaved_tree/broad_leaved_tree_leaves.stl"/>
       </geometry>
     </collision>
@@ -51,8 +51,8 @@
     </inertial>
   </link>
-   <joint name="branch_joint" type="fixed">
+   <joint name="${name}_branch_joint" type="fixed">
     <origin xyz="0 0 0" rpy="0 0 0"/>
     <parent link="${name}"/>
-    <child link="broad_leaved_tree_branches"/>
+    <child link="${name}_branches"/>
   </joint>
     <joint name="${name}_${fixed_frame}_joint"  type="fixed">

File: urdf/conifer.xacro (robot description, xacro)
@@ -10,5 +10,5 @@
       <origin rpy="0 0 0" xyz="0 0 0"/>
       <geometry>
-        <mesh filename="package://iai_outdoor_models/models/broad_leaved_tree/conifer_trunk.stl"/>
+        <mesh filename="package://iai_outdoor_models/models/conifer/conifer_trunk.stl"/>
       </geometry>
       <material name="IAI_RESCUE/broad_leaved_trunk">
@@ -19,5 +19,5 @@
       <origin rpy="0 0 0" xyz="0 0 0"/>
       <geometry>
-        <mesh filename="package://iai_outdoor_models/models/broad_leaved_tree/conifer_trunk.stl"/>
+        <mesh filename="package://iai_outdoor_models/models/conifer/conifer_trunk.stl"/>
       </geometry>
     </collision>
@@ -28,10 +28,10 @@
     </inertial>
   </link>
-  <link name="conifer_branches">
+  <link name="${name}_branches">
     <!--MAIN_BODY-->
     <visual>
       <origin rpy="0 0 0" xyz="0 0 0"/>
       <geometry>
-        <mesh filename="package://iai_outdoor_models/models/broad_leaved_tree/conifer_branches.stl"/>
+        <mesh filename="package://iai_outdoor_models/models/conifer/conifer_branches.stl"/>
       </geometry>
       <material name="IAI_RESCUE/broad_leaved_branch">
@@ -42,5 +42,5 @@
       <origin rpy="0 0 0" xyz="0 0 0"/>
       <geometry>
-        <mesh filename="package://iai_outdoor_models/models/broad_leaved_tree/conifer_branches.stl"/>
+        <mesh filename="package://iai_outdoor_models/models/conifer/conifer_branches.stl"/>
       </geometry>
     </collision>
@@ -51,8 +51,8 @@
     </inertial>
   </link>
-   <joint name="branch_joint" type="fixed">
+   <joint name="${name}_branch_joint" type="fixed">
     <origin xyz="0 0 0" rpy="0 0 0"/>
     <parent link="${name}"/>
-    <child link="conifer_branches"/>
+    <child link="${name}_branches"/>
   </joint>
     <joint name="${name}_${fixed_frame}_joint"  type="fixed">

File: urdf/iai_outdoor_models.xacro (robot description, xacro)
@@ -18,4 +18,8 @@
     <xacro:include filename="$(find iai_outdoor_models)/urdf/conifer.xacro" />
     <xacro:include filename="$(find iai_outdoor_models)/urdf/broad_leaved_tree.xacro" />
+    <xacro:include filename="$(find iai_outdoor_models)/urdf/avalanche_victim.xacro" />
+    <xacro:include filename="$(find iai_outdoor_models)/urdf/lost_victim.xacro" />
+    <xacro:include filename="$(find iai_outdoor_models)/urdf/shoe.xacro" />
+    <xacro:include filename="$(find iai_outdoor_models)/urdf/skis.xacro" />
     <!--
     destroy this one as soon as it is final..

File: urdf/lost_victim.xacro (robot description, xacro)
@@ -1,5 +1,5 @@
 <?xml version="1.0" ?>
-<robot name="rock" xmlns:xacro="http://ros.org/wiki/xacro">
-  <xacro:macro name="rock_macro" params="name fixed_frame *origin">
+<robot name="lost_victim" xmlns:xacro="http://ros.org/wiki/xacro">
+  <xacro:macro name="lost_victim_macro" params="name fixed_frame *origin">
     <gazebo>
       <static>true</static>
@@ -10,5 +10,5 @@
 	<origin rpy="0 0 0" xyz="0 0 0"/>
 	<geometry>
-	  <mesh filename="package://iai_outdoor_models/models/rock/Rock.dae"/>
+	  <mesh filename="package://iai_outdoor_models/models/lost_victim/victim.dae"/>
 	</geometry>
 <!--
@@ -16,5 +16,5 @@
 	-->
 <!--
-	<material name="IAI_RESCUE/rock">
+	<material name="IAI_RESCUE/lost_victim">
 	<color rgba="0.31 0.15 0.033 1.0"/>
       </material>
@@ -24,5 +24,5 @@
 	<origin rpy="0 0 0" xyz="0 0 0"/>
 	<geometry>
-	  <mesh filename="package://iai_outdoor_models/models/rock/Rock.stl"/>
+	  <mesh filename="package://iai_outdoor_models/models/lost_victim/victim.dae"/>
 	</geometry>
       </collision>

File: urdf/shoe.xacro (robot description, xacro)
@@ -1,5 +1,5 @@
 <?xml version="1.0" ?>
-<robot name="rock" xmlns:xacro="http://ros.org/wiki/xacro">
-  <xacro:macro name="rock_macro" params="name fixed_frame *origin">
+<robot name="shoe" xmlns:xacro="http://ros.org/wiki/xacro">
+  <xacro:macro name="shoe_macro" params="name fixed_frame *origin">
     <gazebo>
       <static>true</static>
@@ -10,5 +10,5 @@
 	<origin rpy="0 0 0" xyz="0 0 0"/>
 	<geometry>
-	  <mesh filename="package://iai_outdoor_models/models/rock/Rock.dae"/>
+	  <mesh filename="package://iai_outdoor_models/models/shoe/shoe.dae"/>
 	</geometry>
 <!--
@@ -16,5 +16,5 @@
 	-->
 <!--
-	<material name="IAI_RESCUE/rock">
+	<material name="IAI_RESCUE/shoe">
 	<color rgba="0.31 0.15 0.033 1.0"/>
       </material>
@@ -24,5 +24,5 @@
 	<origin rpy="0 0 0" xyz="0 0 0"/>
 	<geometry>
-	  <mesh filename="package://iai_outdoor_models/models/rock/Rock.stl"/>
+	  <mesh filename="package://iai_outdoor_models/models/shoe/shoe.dae"/>
 	</geometry>
       </collision>

File: urdf/skis.xacro (robot description, xacro)
@@ -1,5 +1,5 @@
 <?xml version="1.0" ?>
-<robot name="rock" xmlns:xacro="http://ros.org/wiki/xacro">
-  <xacro:macro name="rock_macro" params="name fixed_frame *origin">
+<robot name="skis" xmlns:xacro="http://ros.org/wiki/xacro">
+  <xacro:macro name="skis_macro" params="name fixed_frame *origin">
     <gazebo>
       <static>true</static>
@@ -10,5 +10,5 @@
 	<origin rpy="0 0 0" xyz="0 0 0"/>
 	<geometry>
-	  <mesh filename="package://iai_outdoor_models/models/rock/Rock.dae"/>
+	  <mesh filename="package://iai_outdoor_models/models/skis/skis.dae"/>
 	</geometry>
 <!--
@@ -16,5 +16,5 @@
 	-->
 <!--
-	<material name="IAI_RESCUE/rock">
+	<material name="IAI_RESCUE/skis">
 	<color rgba="0.31 0.15 0.033 1.0"/>
       </material>
@@ -24,5 +24,5 @@
 	<origin rpy="0 0 0" xyz="0 0 0"/>
 	<geometry>
-	  <mesh filename="package://iai_outdoor_models/models/rock/Rock.stl"/>
+	  <mesh filename="package://iai_outdoor_models/models/skis/skis.dae"/>
 	</geometry>
       </collision>
